Commit message: ros jazzy + gazebo simulation

File: robots/solo12/xacro/definition.urdf.xacro (robot description, xacro)
@@ -64,9 +64,8 @@
         <material name="solo_grey"><color rgba="0.8 0.8 0.8 1.0"/></material>
       </visual>
-      <collision>
-        <origin xyz="${shoulder_vis_x} 0 0" rpy="0 0 0"/>
-        <geometry>
-          <mesh filename="package://hidro_robots/robots/solo12/meshes/${shoulder_mesh}"/>
-        </geometry>
+      <!-- Simple box collision — mesh trimesh is unstable with ODE/DART -->
+      <collision>
+        <origin xyz="${sh_cx} ${sh_cy} ${sh_cz}" rpy="0 0 0"/>
+        <geometry><box size="0.19 0.035 0.035"/></geometry>
       </collision>
     </link>
@@ -96,9 +95,8 @@
         <material name="solo_grey"><color rgba="0.8 0.8 0.8 1.0"/></material>
       </visual>
-      <collision>
-        <origin xyz="0 0 0" rpy="0 0 0"/>
-        <geometry>
-          <mesh filename="package://hidro_robots/robots/solo12/meshes/${upper_mesh}"/>
-        </geometry>
+      <!-- Simple box collision — mesh trimesh is unstable with ODE/DART -->
+      <collision>
+        <origin xyz="0 0 -0.08" rpy="0 0 0"/>
+        <geometry><box size="0.04 0.04 0.16"/></geometry>
       </collision>
     </link>
@@ -128,9 +126,8 @@
         <material name="solo_grey"><color rgba="0.8 0.8 0.8 1.0"/></material>
       </visual>
-      <collision>
-        <origin xyz="0 0 0" rpy="0 0 0"/>
-        <geometry>
-          <mesh filename="package://hidro_robots/robots/solo12/meshes/${lower_mesh}"/>
-        </geometry>
+      <!-- Sphere at foot tip — approximates ground contact, stable with ODE/DART -->
+      <collision>
+        <origin xyz="0 ${foot_y} -0.155" rpy="0 0 0"/>
+        <geometry><sphere radius="0.020"/></geometry>
       </collision>
     </link>
@@ -188,9 +185,8 @@
         <material name="solo_grey"><color rgba="0.8 0.8 0.8 1.0"/></material>
       </visual>
-      <collision>
-        <origin xyz="0 0 0" rpy="0 0 0"/>
-        <geometry>
-          <mesh filename="package://hidro_robots/robots/solo12/meshes/solo_12_base.stl"/>
-        </geometry>
+      <!-- Simple box collision — mesh trimesh is unstable with ODE/DART -->
+      <collision>
+        <origin xyz="0 0 0" rpy="0 0 0"/>
+        <geometry><box size="0.25 0.15 0.04"/></geometry>
       </collision>
     </link>
@@ -266,5 +262,5 @@
       <xacro:unless value="${event_based_sim}">
         <gazebo>
-          <plugin name="odri_gazebo" filename="libodri_gazebo_plugin.so">
+          <plugin name="odri_ros2_gazebo_plugin::OdriGazeboPlugin" filename="libodri_gazebo_plugin.so">
             <joint name="FL_HAA"><param name="safe_position"> 0.0</param><param name="safe_torque">0.5</param></joint>
             <joint name="FL_HFE"><param name="safe_position"> 0.8</param><param name="safe_torque">0.5</param></joint>
